File: matrix.sch (KiCad schematic (older format))
At the start: 17 parts, among them Y1 16MHz

Commit message: corefix
Parts:
- removed C3: 0.1uF, symbol Device:C_Small
- gave numbers to parts that had none: 1
Connections:
- net +5V: now also C2.1, U?.8 (VBUS); no longer C2.2
- net GND: now also C1.2, C2.2
Other:
- moved on the sheet: C2

Commit message: typecadd
Parts:
- added F1: 500m, symbol Device:Polyfuse_Small
- added J1: AVR-ISP-6, symbol Connector:AVR-ISP-6
- added R4, R?: 5.1k, symbol Device:R_Small_US
- added U2: PRTR5V0U2X, symbol random-keyboard-parts:PRTR5V0U2X
- added USBC: HRO-TYPE-C-31-M-12, symbol Type-C:HRO-TYPE-C-31-M-12
- gave numbers to parts that had none: 1
Connections:
- net +5V: now also F1.1, J1.6 (GND)
- net D+: now also U2.2 (IO1), USBC.6 (DP1), USBC.8 (DP2)
- net D-: now also U2.3 (IO2), USBC.5 (DN2), USBC.7 (DN1)
- net GND: now also J1.2 (VCC), R4.1, R?.1, U2.1 (GND), USBC.1 (GND), USBC.12 (GND), USBC.13 (SHIELD)
- net SCLK: now reaches U1.11 (PB1)
- net SCLK: now also J1.3 (SCK)
- net MOSI: now reaches U1.12 (PB2)
- net MOSI: now also J1.4 (MOSI)
- net MISO: now reaches U1.13 (PB3)
- net MISO: now also J1.1 (MISO)
- net RESET: now reaches 10k.2, Reset.2, U1.20 (~RESET)
- net RESET: now also J1.5 (~RST)
- new net: R4.2, USBC.10 (CC2)
- new net: R?.2, USBC.4 (CC1)
- new net VCC: F1.2, U2.4 (VCC), USBC.11 (VBUS), USBC.2 (VBUS)
- no-connect marks 0 -> 2
Other:
- moved on the sheet: 10k, Reset

Commit message: schematicfootprintless
Parts:
- added SW1, SW2: Rotary_Encoder, symbol Device:Rotary_Encoder
- R3: renamed from 10k; value R3 -> 10k
- gave numbers to parts that had none: 1
- renumbered C3 to C30, C3 to C31, C3 to C32, C3 to C33, C3 to C34, C4 to C40, C4 to C41, R2 to R20, R2 to R21, R4 to R40, Reset to Reset1, USBC to USBC1
Connections:
- net D+: now also R20.1, U1.5 (D+); no longer R21.2, U2.2 (IO1), USBC1.6 (DP1), USBC1.8 (DP2)
- net D-: now also R21.1, U1.4 (D-); no longer R20.2, U2.3 (IO2), USBC1.5 (DN2), USBC1.7 (DN1)
- net GND: now also SW1.C, SW2.C
- net COL9: now reaches U1.1 (PE6)
- net COL6: now reaches U1.10 (PB0)
- net COL5: now reaches U1.14 (PB4)
- net COL4: now reaches U1.15 (PB5)
- net COL3: now reaches U1.16 (PB6)
- net COL2: now reaches U1.17 (PB7)
- net COL1: now reaches U1.18 (PE4)
- net COL0: now reaches U1.19 (PE5)
- net COL8: now reaches U1.2 (PE7)
- net XTAL2: now reaches C41.1, U1.23 (XTAL2), Y1.2
- net XTAL1: now reaches C40.1, U1.24 (XTAL1), Y1.4
- net ROW0: now reaches U1.25 (PD0)
- net ROW1: now reaches U1.26 (PD1)
- net ROW2: now reaches U1.27 (PD2)
- net ROW3: now reaches U1.28 (PD3)
- net ROW4: now reaches U1.29 (PD4)
- net ROW5: now reaches U1.30 (PD5)
- net COL16: now reaches U1.55 (PF6)
- net COL15: now reaches U1.56 (PF5)
- net COL14: now reaches U1.57 (PF4)
- net COL13: now reaches U1.58 (PF3)
- net COL12: now reaches U1.59 (PF2)
- net COL11: now reaches U1.60 (PF1)
- net COL10: now reaches U1.61 (PF0)
- net COL7: now reaches U1.9 (PE3)
- new net: R21.2, U2.3 (IO2), USBC1.5 (DN2), USBC1.7 (DN1)
- new net: R20.2, U2.2 (IO1), USBC1.6 (DP1), USBC1.8 (DP2)
- new net R00: SW2.A
- new net R01: SW2.B
- new net R10: SW1.A
- new net R11: SW1.B
- no-connect marks 2 -> 24
Other:
- moved on the sheet: C1, C2, C30, C31, C32, C33, C34, C40, C41, F1, J1, R1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
