File: matrix.sch (KiCad schematic (older format))
At the start: 24 parts, among them J1 AVR-ISP-6, SW1 Rotary_Encoder, SW2 Rotary_Encoder, U1 AT90USB1286-AU, U2 PRTR5V0U2X, Y1 16MHz

Commit message: footprints
Parts:
- C1, C2, C30, C31, C32, C33, C34, C40, C41: footprint (none) -> Capacitor_SMD:C_1206_3216Metric_Pad1.42x1.75mm_HandSolder
- F1: footprint (none) -> Fuse:Fuse_1206_3216Metric_Pad1.42x1.75mm_HandSolder
- J1: footprint (none) -> random-keyboard-parts:Reset_Pretty-Mask
- R1, R20, R21, R3, R40, R41: footprint (none) -> Resistor_SMD:R_1206_3216Metric_Pad1.42x1.75mm_HandSolder
- Reset1: footprint (none) -> Button_Switch_SMD:SW_SPST_SKQG_WithStem
- SW1, SW2: footprint (none) -> Rotary_Encoder:RotaryEncoder_Alps_EC11E_Vertical_H20mm
- U2: footprint (none) -> random-keyboard-parts:SOT143B
- USBC1: footprint (none) -> Type-C:HRO-TYPE-C-31-M-12-HandSoldering
- Y1: footprint (none) -> Crystal:Crystal_SMD_3225-4Pin_3.2x2.5mm_HandSoldering
Changed lines of the file:
@@
 F 0 "R1" V 12095 6050 50  0000 C CNN
 F 1 "1k" V 12186 6050 50  0000 C CNN
-F 2 "" H 12300 6050 50  0001 C CNN
+F 2 "Resistor_SMD:R_1206_3216Metric_Pad1.42x1.75mm_HandSolder" H 12300 6050 50  0001 C CNN
 F 3 "~" H 12300 6050 50  0001 C CNN
 	1    12300 6050
@@
 F 0 "C1" V 12021 5350 50  0000 C CNN
 F 1 "1uF" V 12112 5350 50  0000 C CNN
-F 2 "" H 12250 5350 50  0001 C CNN
+F 2 "Capacitor_SMD:C_1206_3216Metric_Pad1.42x1.75mm_HandSolder" H 12250 5350 50  0001 C CNN
 F 3 "~" H 12250 5350 50  0001 C CNN
 	1    12250 5350
@@
 F 0 "C31" H 14942 3596 50  0000 L CNN
 F 1 "0.1uF" H 14942 3505 50  0000 L CNN
-F 2 "" H 14850 3550 50  0001 C CNN
+F 2 "Capacitor_SMD:C_1206_3216Metric_Pad1.42x1.75mm_HandSolder" H 14850 3550 50  0001 C CNN
 F 3 "~" H 14850 3550 50  0001 C CNN
 	1    14850 3550
@@
 F 0 "C32" H 15342 3596 50  0000 L CNN
 F 1 "0.1uF" H 15342 3505 50  0000 L CNN
-F 2 "" H 15250 3550 50  0001 C CNN
+F 2 "Capacitor_SMD:C_1206_3216Metric_Pad1.42x1.75mm_HandSolder" H 15250 3550 50  0001 C CNN
 F 3 "~" H 15250 3550 50  0001 C CNN
 	1    15250 3550
@@
 F 0 "C33" H 15742 3596 50  0000 L CNN
 F 1 "0.1uF" H 15742 3505 50  0000 L CNN
-F 2 "" H 15650 3550 50  0001 C CNN
+F 2 "Capacitor_SMD:C_1206_3216Metric_Pad1.42x1.75mm_HandSolder" H 15650 3550 50  0001 C CNN
 F 3 "~" H 15650 3550 50  0001 C CNN
 	1    15650 3550
@@
 F 0 "C34" H 16142 3596 50  0000 L CNN
 F 1 "0.1uF" H 16142 3505 50  0000 L CNN
-F 2 "" H 16050 3550 50  0001 C CNN
+F 2 "Capacitor_SMD:C_1206_3216Metric_Pad1.42x1.75mm_HandSolder" H 16050 3550 50  0001 C CNN
 F 3 "~" H 16050 3550 50  0001 C CNN
 	1    16050 3550
@@
 F 0 "C30" H 14542 3596 50  0000 L CNN
 F 1 "0.1uF" H 14542 3505 50  0000 L CNN
-F 2 "" H 14450 3550 50  0001 C CNN
+F 2 "Capacitor_SMD:C_1206_3216Metric_Pad1.42x1.75mm_HandSolder" H 14450 3550 50  0001 C CNN
 F 3 "~" H 14450 3550 50  0001 C CNN
 	1    14450 3550
@@
 F 0 "Y1" H 14944 7796 50  0000 L CNN
 F 1 "16MHz" H 14944 7705 50  0000 L CNN
-F 2 "" H 14800 7750 50  0001 C CNN
+F 2 "Crystal:Crystal_SMD_3225-4Pin_3.2x2.5mm_HandSoldering" H 14800 7750 50  0001 C CNN
 F 3 "~" H 14800 7750 50  0001 C CNN
 	1    14800 7750
@@
 F 0 "C40" V 14271 7550 50  0000 C CNN
 F 1 "22pF" V 14362 7550 50  0000 C CNN
-F 2 "" H 14500 7550 50  0001 C CNN
+F 2 "Capacitor_SMD:C_1206_3216Metric_Pad1.42x1.75mm_HandSolder" H 14500 7550 50  0001 C CNN
 F 3 "~" H 14500 7550 50  0001 C CNN
 	1    14500 7550
@@
 F 0 "C41" V 14271 7950 50  0000 C CNN
 F 1 "22pF" V 14362 7950 50  0000 C CNN
-F 2 "" H 14500 7950 50  0001 C CNN
+F 2 "Capacitor_SMD:C_1206_3216Metric_Pad1.42x1.75mm_HandSolder" H 14500 7950 50  0001 C CNN
 F 3 "~" H 14500 7950 50  0001 C CNN
 	1    14500 7950
@@
 F 0 "R3" H 16018 4396 50  0000 L CNN
 F 1 "10k" H 16018 4305 50  0000 L CNN
-F 2 "" H 15950 4350 50  0001 C CNN
+F 2 "Resistor_SMD:R_1206_3216Metric_Pad1.42x1.75mm_HandSolder" H 15950 4350 50  0001 C CNN
 F 3 "~" H 15950 4350 50  0001 C CNN
 	1    15950 4350
@@
 F 0 "Reset1" H 15650 4485 50  0000 C CNN
 F 1 "SW_Push" H 15650 4394 50  0000 C CNN
-F 2 "" H 15650 4400 50  0001 C CNN
+F 2 "Button_Switch_SMD:SW_SPST_SKQG_WithStem" H 15650 4400 50  0001 C CNN
 F 3 "~" H 15650 4400 50  0001 C CNN
 	1    15650 4200
@@
 F 0 "C2" V 13821 3550 50  0000 C CNN
 F 1 "10uF" V 13912 3550 50  0000 C CNN
-F 2 "" H 14050 3550 50  0001 C CNN
+F 2 "Capacitor_SMD:C_1206_3216Metric_Pad1.42x1.75mm_HandSolder" H 14050 3550 50  0001 C CNN
 F 3 "~" H 14050 3550 50  0001 C CNN
 	1    14050 3550
@@
 F 0 "USBC1" H 14833 6747 60  0000 C CNN
 F 1 "HRO-TYPE-C-31-M-12" H 14833 6641 60  0000 C CNN
-F 2 "" H 15000 5950 60  0001 C CNN
+F 2 "Type-C:HRO-TYPE-C-31-M-12-HandSoldering" H 15000 5950 60  0001 C CNN
 F 3 "" H 15000 5950 60  0001 C CNN
 	1    15000 5950
@@
 F 0 "F1" V 15695 5500 50  0000 C CNN
 F 1 "500m" V 15786 5500 50  0000 C CNN
-F 2 "" H 15950 5300 50  0001 L CNN
+F 2 "Fuse:Fuse_1206_3216Metric_Pad1.42x1.75mm_HandSolder" H 15950 5300 50  0001 L CNN
 F 3 "~" H 15900 5500 50  0001 C CNN
 	1    15900 5500
@@
 F 0 "R41" V 15095 5700 50  0000 C CNN
 F 1 "5.1k" V 15186 5700 50  0000 C CNN
-F 2 "" H 15300 5700 50  0001 C CNN
+F 2 "Resistor_SMD:R_1206_3216Metric_Pad1.42x1.75mm_HandSolder" H 15300 5700 50  0001 C CNN
 F 3 "~" H 15300 5700 50  0001 C CNN
 	1    15300 5700
@@
 F 0 "R40" V 15095 6300 50  0000 C CNN
 F 1 "5.1k" V 15186 6300 50  0000 C CNN
-F 2 "" H 15300 6300 50  0001 C CNN
+F 2 "Resistor_SMD:R_1206_3216Metric_Pad1.42x1.75mm_HandSolder" H 15300 6300 50  0001 C CNN
 F 3 "~" H 15300 6300 50  0001 C CNN
 	1    15300 6300
@@
 F 0 "U2" H 14750 6713 60  0000 C CNN
 F 1 "PRTR5V0U2X" H 14750 6819 60  0000 C CNN
-F 2 "" H 14750 7000 60  0001 C CNN
+F 2 "random-keyboard-parts:SOT143B" H 14750 7000 60  0001 C CNN
 F 3 "" H 14750 7000 60  0001 C CNN
 	1    14750 7000
@@
 F 0 "J1" H 14420 4304 50  0000 R CNN
 F 1 "AVR-ISP-6" H 14420 4395 50  0000 R CNN
-F 2 "" V 14450 4350 50  0001 C CNN
+F 2 "random-keyboard-parts:Reset_Pretty-Mask" V 14450 4350 50  0001 C CNN
 F 3 " ~" H 13425 3750 50  0001 C CNN
 	1    14700 4300
@@
 F 0 "R20" V 15745 6100 50  0000 C CNN
 F 1 "22" V 15836 6100 50  0000 C CNN
-F 2 "" H 15950 6100 50  0001 C CNN
+F 2 "Resistor_SMD:R_1206_3216Metric_Pad1.42x1.75mm_HandSolder" H 15950 6100 50  0001 C CNN
 F 3 "~" H 15950 6100 50  0001 C CNN
 	1    15950 6100
@@
 F 0 "R21" V 15545 6000 50  0000 C CNN
 F 1 "22" V 15636 6000 50  0000 C CNN
-F 2 "" H 15750 6000 50  0001 C CNN
+F 2 "Resistor_SMD:R_1206_3216Metric_Pad1.42x1.75mm_HandSolder" H 15750 6000 50  0001 C CNN
 F 3 "~" H 15750 6000 50  0001 C CNN
 	1    15750 6000
@@
 F 0 "SW1" H 15380 8996 50  0000 L CNN
 F 1 "Rotary_Encoder" H 15380 8905 50  0000 L CNN
-F 2 "" H 15000 9110 50  0001 C CNN
+F 2 "Rotary_Encoder:RotaryEncoder_Alps_EC11E_Vertical_H20mm" H 15000 9110 50  0001 C CNN
 F 3 "~" H 15150 9210 50  0001 C CNN
 	1    15150 8950
@@
 F 0 "SW2" H 15380 8546 50  0000 L CNN
 F 1 "Rotary_Encoder" H 15380 8455 50  0000 L CNN
-F 2 "" H 15000 8660 50  0001 C CNN
+F 2 "Rotary_Encoder:RotaryEncoder_Alps_EC11E_Vertical_H20mm" H 15000 8660 50  0001 C CNN
 F 3 "~" H 15150 8760 50  0001 C CNN
 	1    15150 8500

Commit message: ithinkdoneschematic
Connections:
- net RGB: now reaches U1.54 (PF7)
- no-connect marks 20 -> 19
Changed lines of the file:
@@
 $Descr User 17000 11000
 encoding utf-8
-Sheet 1 2
+Sheet 1 3
 Title ""
 Date ""
@@
 Comment4 ""
 $EndDescr
-$Sheet
-S 800  650  11100 9550
-U 6547D7EB
-F0 "keymatrix" 50
-F1 "keymatrix.sch" 50
-$EndSheet
 Text Notes 12650 10250 0    50   ~ 0
 Matrix MK. I
@@
 Text GLabel 16100 4450 2    50   Input ~ 0
 RESET
-NoConn ~ 12650 7450
 NoConn ~ 12650 4650
 NoConn ~ 13850 6550
@@
 Text GLabel 12650 5950 0    50   Input ~ 0
 R11
+$Sheet
+S 800  650  6000 9750
+U 6547D7EB
+F0 "keymatrix" 50
+F1 "keymatrix.sch" 50
+$EndSheet
+$Sheet
+S 7300 700  4550 9600
+U 654946C7
+F0 "matrixrgb" 50
+F1 "matrixrgb.sch" 50
+$EndSheet
+Text GLabel 12650 7450 0    50   Input ~ 0
+RGB
 $EndSCHEMATC

Commit message: prerouting+finalnewdoneschematicIswear
Parts:
- added C1: 0.1uF, Capacitor_SMD:C_1206_3216Metric_Pad1.42x1.75mm_HandSolder, symbol Device:C_Small
- added C2: 1uF, Capacitor_SMD:C_1206_3216Metric_Pad1.42x1.75mm_HandSolder, symbol Device:C_Small
- added D1, D10, D11, D12, D13, D14, D15, D16, D17, D18, D19, D2, D20, D21, D22, D23, D24, D25, D26, D27, D28, D29, D3, D30, D31, D32, D33, D34, D35, D36, D37, D38, D39, D4, D40, D41, D42, D43, D44, D45, D46, D47, D48, D49, D5, D50, D51, D52, D53, D54, D55, D56, D57, D58, D59, D6, D60, D61, D62, D63, D64, D65, D66, D67, D68, D69, D7, D70, D71, D72, D73, D74, D75, D76, D77, D78, D79, D8, D80, D81, D82, D83, D84, D85, D86, D87, D88, D9: D, Diode_SMD:D_SOD-123, symbol Device:D
- added D100, D101, D102, D103, D104, D105, D106, D107, D108, D109, D110, D111, D112, D113, D114, D115, D116, D117, D118, D119, D120, D121, D122, D123, D124, D125, D126, D127, D128, D129, D130, D131, D132, D133, D134, D135, D136, D137, D138, D139, D140, D141, D142, D143, D144, D145, D146, D147, D148, D149, D150, D151, D152, D153, D154, D155, D156, D157, D158, D159, D160, D161, D162, D163, D164, D165, D166, D167, D168, D169, D170, D171, D172, D173, D174, D175, D176, D177, D178, D190, D191, D89, D90, D91, D92, D93, D94, D95, D96, D97, D98, D99: LED, LED_SMD:LED_1206_3216Metric_ReverseMount_Hole1.8x2.4mm, symbol Device:LED
- added MX1: ESC, MX_Alps_Hybrid:MX-1U-NoLED, symbol MX_Alps_Hybrid:MX-NoLED
- added MX10: F9, MX_Alps_Hybrid:MX-1U-NoLED, symbol MX_Alps_Hybrid:MX-NoLED
- added MX11: F10, MX_Alps_Hybrid:MX-1U-NoLED, symbol MX_Alps_Hybrid:MX-NoLED
- added MX12: F11, MX_Alps_Hybrid:MX-1U-NoLED, symbol MX_Alps_Hybrid:MX-NoLED
- added MX13: F12, MX_Alps_Hybrid:MX-1U-NoLED, symbol MX_Alps_Hybrid:MX-NoLED
- added MX14: HOME, MX_Alps_Hybrid:MX-1U-NoLED, symbol MX_Alps_Hybrid:MX-NoLED
- added MX15: END, MX_Alps_Hybrid:MX-1U-NoLED, symbol MX_Alps_Hybrid:MX-NoLED
- added MX16: INSERT, MX_Alps_Hybrid:MX-1U-NoLED, symbol MX_Alps_Hybrid:MX-NoLED
- added MX17: MCRO1, MX_Alps_Hybrid:MX-1U-NoLED, symbol MX_Alps_Hybrid:MX-NoLED
- added MX18: ,~, MX_Alps_Hybrid:MX-1U-NoLED, symbol MX_Alps_Hybrid:MX-NoLED
- added MX19: 1!, MX_Alps_Hybrid:MX-1U-NoLED, symbol MX_Alps_Hybrid:MX-NoLED
- added MX2: F1, MX_Alps_Hybrid:MX-1U-NoLED, symbol MX_Alps_Hybrid:MX-NoLED
- added MX20: 2@, MX_Alps_Hybrid:MX-1U-NoLED, symbol MX_Alps_Hybrid:MX-NoLED
- added MX21: 3#, MX_Alps_Hybrid:MX-1U-NoLED, symbol MX_Alps_Hybrid:MX-NoLED
- added MX22: 4$, MX_Alps_Hybrid:MX-1U-NoLED, symbol MX_Alps_Hybrid:MX-NoLED
- added MX23: 5%, MX_Alps_Hybrid:MX-1U-NoLED, symbol MX_Alps_Hybrid:MX-NoLED
- added MX24: 6^, MX_Alps_Hybrid:MX-1U-NoLED, symbol MX_Alps_Hybrid:MX-NoLED
- added MX25: 7&, MX_Alps_Hybrid:MX-1U-NoLED, symbol MX_Alps_Hybrid:MX-NoLED
- added MX26: 8*, MX_Alps_Hybrid:MX-1U-NoLED, symbol MX_Alps_Hybrid:MX-NoLED
- added MX27: 9(, MX_Alps_Hybrid:MX-1U-NoLED, symbol MX_Alps_Hybrid:MX-NoLED
- added MX28: 0), MX_Alps_Hybrid:MX-1U-NoLED, symbol MX_Alps_Hybrid:MX-NoLED
- added MX29: -_, MX_Alps_Hybrid:MX-1U-NoLED, symbol MX_Alps_Hybrid:MX-NoLED
- added MX3: F2, MX_Alps_Hybrid:MX-1U-NoLED, symbol MX_Alps_Hybrid:MX-NoLED
- added MX30: =+, MX_Alps_Hybrid:MX-1U-NoLED, symbol MX_Alps_Hybrid:MX-NoLED
- added MX31: BCSP, MX_Alps_Hybrid:MX-2U-NoLED, symbol MX_Alps_Hybrid:MX-NoLED
- added MX32: DEL, MX_Alps_Hybrid:MX-1U-NoLED, symbol MX_Alps_Hybrid:MX-NoLED
- added MX33: MCRO2, MX_Alps_Hybrid:MX-1U-NoLED, symbol MX_Alps_Hybrid:MX-NoLED
- added MX34: TABL, MX_Alps_Hybrid:MX-1.5U-NoLED, symbol MX_Alps_Hybrid:MX-NoLED
- added MX35: Q, MX_Alps_Hybrid:MX-1U-NoLED, symbol MX_Alps_Hybrid:MX-NoLED
- added MX36: W, MX_Alps_Hybrid:MX-1U-NoLED, symbol MX_Alps_Hybrid:MX-NoLED
- added MX37: E, MX_Alps_Hybrid:MX-1U-NoLED, symbol MX_Alps_Hybrid:MX-NoLED
- added MX38: R, MX_Alps_Hybrid:MX-1U-NoLED, symbol MX_Alps_Hybrid:MX-NoLED
- added MX39: T, MX_Alps_Hybrid:MX-1U-NoLED, symbol MX_Alps_Hybrid:MX-NoLED
- added MX4: F3, MX_Alps_Hybrid:MX-1U-NoLED, symbol MX_Alps_Hybrid:MX-NoLED
- added MX40: Y, MX_Alps_Hybrid:MX-1U-NoLED, symbol MX_Alps_Hybrid:MX-NoLED
- added MX41: U, MX_Alps_Hybrid:MX-1U-NoLED, symbol MX_Alps_Hybrid:MX-NoLED
- added MX42: I, MX_Alps_Hybrid:MX-1U-NoLED, symbol MX_Alps_Hybrid:MX-NoLED
- added MX43: O, MX_Alps_Hybrid:MX-1U-NoLED, symbol MX_Alps_Hybrid:MX-NoLED
- added MX44: P, MX_Alps_Hybrid:MX-1U-NoLED, symbol MX_Alps_Hybrid:MX-NoLED
- added MX45: [{, MX_Alps_Hybrid:MX-1U-NoLED, symbol MX_Alps_Hybrid:MX-NoLED
- added MX46: ]}, MX_Alps_Hybrid:MX-1U-NoLED, symbol MX_Alps_Hybrid:MX-NoLED
- added MX47: \\|, MX_Alps_Hybrid:MX-1.5U-NoLED, symbol MX_Alps_Hybrid:MX-NoLED
- added MX48: PGUP, MX_Alps_Hybrid:MX-1U-NoLED, symbol MX_Alps_Hybrid:MX-NoLED
- added MX49: MCRO3, MX_Alps_Hybrid:MX-1U-NoLED, symbol MX_Alps_Hybrid:MX-NoLED
- added MX5: F4, MX_Alps_Hybrid:MX-1U-NoLED, symbol MX_Alps_Hybrid:MX-NoLED
- added MX50: CPLK, MX_Alps_Hybrid:MX-1.75U-NoLED, symbol MX_Alps_Hybrid:MX-NoLED
- added MX51: A, MX_Alps_Hybrid:MX-1U-NoLED, symbol MX_Alps_Hybrid:MX-NoLED
- added MX52: S, MX_Alps_Hybrid:MX-1U-NoLED, symbol MX_Alps_Hybrid:MX-NoLED
- added MX53: D, MX_Alps_Hybrid:MX-1U-NoLED, symbol MX_Alps_Hybrid:MX-NoLED
- added MX54: F, MX_Alps_Hybrid:MX-1U-NoLED, symbol MX_Alps_Hybrid:MX-NoLED
- added MX55: G, MX_Alps_Hybrid:MX-1U-NoLED, symbol MX_Alps_Hybrid:MX-NoLED
- added MX56: H, MX_Alps_Hybrid:MX-1U-NoLED, symbol MX_Alps_Hybrid:MX-NoLED
- added MX57: J, MX_Alps_Hybrid:MX-1U-NoLED, symbol MX_Alps_Hybrid:MX-NoLED
- added MX58: K, MX_Alps_Hybrid:MX-1U-NoLED, symbol MX_Alps_Hybrid:MX-NoLED
- added MX59: L, MX_Alps_Hybrid:MX-1U-NoLED, symbol MX_Alps_Hybrid:MX-NoLED
- added MX6: F5, MX_Alps_Hybrid:MX-1U-NoLED, symbol MX_Alps_Hybrid:MX-NoLED
- added MX60: ;:, MX_Alps_Hybrid:MX-1U-NoLED, symbol MX_Alps_Hybrid:MX-NoLED
- added MX61: '\", MX_Alps_Hybrid:MX-1U-NoLED, symbol MX_Alps_Hybrid:MX-NoLED
- added MX62: ENTR, MX_Alps_Hybrid:MX-2.25U-NoLED, symbol MX_Alps_Hybrid:MX-NoLED
- added MX63: PGDN, MX_Alps_Hybrid:MX-1U-NoLED, symbol MX_Alps_Hybrid:MX-NoLED
- added MX64: MCRO4, MX_Alps_Hybrid:MX-1U-NoLED, symbol MX_Alps_Hybrid:MX-NoLED
- added MX65: SHIFTL, MX_Alps_Hybrid:MX-2.25U-NoLED, symbol MX_Alps_Hybrid:MX-NoLED
- added MX66: Z, MX_Alps_Hybrid:MX-1U-NoLED, symbol MX_Alps_Hybrid:MX-NoLED
- added MX67: X, MX_Alps_Hybrid:MX-1U-NoLED, symbol MX_Alps_Hybrid:MX-NoLED
- added MX68: C, MX_Alps_Hybrid:MX-1U-NoLED, symbol MX_Alps_Hybrid:MX-NoLED
- added MX69: V, MX_Alps_Hybrid:MX-1U-NoLED, symbol MX_Alps_Hybrid:MX-NoLED
- added MX7: F6, MX_Alps_Hybrid:MX-1U-NoLED, symbol MX_Alps_Hybrid:MX-NoLED
- added MX70: B, MX_Alps_Hybrid:MX-1U-NoLED, symbol MX_Alps_Hybrid:MX-NoLED
- added MX71: N, MX_Alps_Hybrid:MX-1U-NoLED, symbol MX_Alps_Hybrid:MX-NoLED
- added MX72: M, MX_Alps_Hybrid:MX-1U-NoLED, symbol MX_Alps_Hybrid:MX-NoLED
- added MX73: ,<, MX_Alps_Hybrid:MX-1U-NoLED, symbol MX_Alps_Hybrid:MX-NoLED
- added MX74: .>, MX_Alps_Hybrid:MX-1U-NoLED, symbol MX_Alps_Hybrid:MX-NoLED
- added MX75: /?, MX_Alps_Hybrid:MX-1U-NoLED, symbol MX_Alps_Hybrid:MX-NoLED
- added MX76: SHIFTR, MX_Alps_Hybrid:MX-2.75U-NoLED, symbol MX_Alps_Hybrid:MX-NoLED
- added MX77: UP, MX_Alps_Hybrid:MX-1U-NoLED, symbol MX_Alps_Hybrid:MX-NoLED
- added MX78: CTRLL, MX_Alps_Hybrid:MX-1.25U-NoLED, symbol MX_Alps_Hybrid:MX-NoLED
- added MX79: WIN, MX_Alps_Hybrid:MX-1.25U-NoLED, symbol MX_Alps_Hybrid:MX-NoLED
- added MX8: F7, MX_Alps_Hybrid:MX-1U-NoLED, symbol MX_Alps_Hybrid:MX-NoLED
- added MX80: ALTL, MX_Alps_Hybrid:MX-1.25U-NoLED, symbol MX_Alps_Hybrid:MX-NoLED
- added MX81: SPCB, MX_Alps_Hybrid:MX-6.25U-NoLED, symbol MX_Alps_Hybrid:MX-NoLED
- added MX82: ALTR, MX_Alps_Hybrid:MX-1U-NoLED, symbol MX_Alps_Hybrid:MX-NoLED
- added MX83: MENU, MX_Alps_Hybrid:MX-1U-NoLED, symbol MX_Alps_Hybrid:MX-NoLED
- added MX84: FN, MX_Alps_Hybrid:MX-1U-NoLED, symbol MX_Alps_Hybrid:MX-NoLED
- added MX85: CTRLR, MX_Alps_Hybrid:MX-1U-NoLED, symbol MX_Alps_Hybrid:MX-NoLED
- added MX86: LEFT, MX_Alps_Hybrid:MX-1U-NoLED, symbol MX_Alps_Hybrid:MX-NoLED
- added MX87: DOWN, MX_Alps_Hybrid:MX-1U-NoLED, symbol MX_Alps_Hybrid:MX-NoLED
- added MX88: RIGHT, MX_Alps_Hybrid:MX-1U-NoLED, symbol MX_Alps_Hybrid:MX-NoLED
- added MX9: F8, MX_Alps_Hybrid:MX-1U-NoLED, symbol MX_Alps_Hybrid:MX-NoLED
- added R1, R2: 4k7, Resistor_SMD:R_1206_3216Metric_Pad1.42x1.75mm_HandSolder, symbol Device:R_Small_US
- added R11, R12: 470, Resistor_SMD:R_1206_3216Metric_Pad1.42x1.75mm_HandSolder, symbol Device:R_Small_US
- added R3: 100k, Resistor_SMD:R_1206_3216Metric_Pad1.42x1.75mm_HandSolder, symbol Device:R_Small_US
- added R4: 20k, Resistor_SMD:R_1206_3216Metric_Pad1.42x1.75mm_HandSolder, symbol Device:R_Small_US
- added U1: IS31FL3731-SA, Package_SO:SSOP-28_5.3x10.2mm_P0.65mm, symbol Driver_LED:IS31FL3731-SA
- renumbered C40 to C10, C41 to C11, C2 to C3, C30 to C4, C31 to C5, C32 to C6, C33 to C7, C34 to C8, C1 to C9, R40 to R10, R3 to R5, R41 to R6, R21 to R7, R1 to R8, R20 to R9, SW2 to SW1, SW1 to SW2, U1 to U2, U2 to U3
Connections:
- net COL0: now also MX1.1 (COL), MX18.1 (COL), MX34.1 (COL), MX50.1 (COL), MX78.1 (COL)
- net COL1: now also MX19.1 (COL), MX2.1 (COL), MX65.1 (COL), MX79.1 (COL)
- net COL10: now also MX11.1 (COL), MX28.1 (COL), MX43.1 (COL), MX59.1 (COL), MX74.1 (COL), MX82.1 (COL)
- net COL11: now also MX12.1 (COL), MX29.1 (COL), MX44.1 (COL), MX60.1 (COL), MX75.1 (COL), MX83.1 (COL)
- net COL12: now also MX13.1 (COL), MX30.1 (COL), MX45.1 (COL), MX61.1 (COL), MX84.1 (COL)
- net COL13: now also MX14.1 (COL), MX46.1 (COL), MX62.1 (COL), MX76.1 (COL), MX85.1 (COL)
- net COL14: now also MX15.1 (COL), MX31.1 (COL), MX47.1 (COL), MX86.1 (COL)
- net COL15: now also MX16.1 (COL), MX32.1 (COL), MX48.1 (COL), MX63.1 (COL), MX77.1 (COL), MX87.1 (COL)
- net COL16: now also MX17.1 (COL), MX33.1 (COL), MX49.1 (COL), MX64.1 (COL), MX88.1 (COL)
- net COL2: now also MX20.1 (COL), MX3.1 (COL), MX35.1 (COL), MX51.1 (COL), MX66.1 (COL)
- net COL3: now also MX21.1 (COL), MX36.1 (COL), MX4.1 (COL), MX52.1 (COL), MX67.1 (COL), MX80.1 (COL)
- net COL4: now also MX22.1 (COL), MX37.1 (COL), MX5.1 (COL), MX53.1 (COL), MX68.1 (COL)
- net COL5: now also MX23.1 (COL), MX38.1 (COL), MX54.1 (COL), MX6.1 (COL), MX69.1 (COL)
- net COL6: now also MX24.1 (COL), MX39.1 (COL), MX55.1 (COL), MX7.1 (COL), MX70.1 (COL), MX81.1 (COL)
- net COL7: now also MX25.1 (COL), MX40.1 (COL), MX56.1 (COL), MX71.1 (COL), MX8.1 (COL)
- net COL8: now also MX26.1 (COL), MX41.1 (COL), MX57.1 (COL), MX72.1 (COL), MX9.1 (COL)
- net COL9: now also MX10.1 (COL), MX27.1 (COL), MX42.1 (COL), MX58.1 (COL), MX73.1 (COL)
- net GND: now also C1.2, C2.2, R11.1, R12.1, R3.2, R4.1, U1.18 (AD), U1.5 (GND)
- net ROW0: now also D1.1 (K), D10.1 (K), D11.1 (K), D12.1 (K), D13.1 (K), D14.1 (K), D15.1 (K), D16.1 (K), D17.1 (K), D2.1 (K), D3.1 (K), D4.1 (K), D5.1 (K), D6.1 (K), D7.1 (K), D8.1 (K), D9.1 (K)
- net ROW1: now also D18.1 (K), D19.1 (K), D20.1 (K), D21.1 (K), D22.1 (K), D23.1 (K), D24.1 (K), D25.1 (K), D26.1 (K), D27.1 (K), D28.1 (K), D29.1 (K), D30.1 (K), D31.1 (K), D32.1 (K), D33.1 (K)
- net ROW2: now also D34.1 (K), D35.1 (K), D36.1 (K), D37.1 (K), D38.1 (K), D39.1 (K), D40.1 (K), D41.1 (K), D42.1 (K), D43.1 (K), D44.1 (K), D45.1 (K), D46.1 (K), D47.1 (K), D48.1 (K), D49.1 (K)
- net ROW3: now also D50.1 (K), D51.1 (K), D52.1 (K), D53.1 (K), D54.1 (K), D55.1 (K), D56.1 (K), D57.1 (K), D58.1 (K), D59.1 (K), D60.1 (K), D61.1 (K), D62.1 (K), D63.1 (K), D64.1 (K)
- net ROW4: now also D65.1 (K), D66.1 (K), D67.1 (K), D68.1 (K), D69.1 (K), D70.1 (K), D71.1 (K), D72.1 (K), D73.1 (K), D74.1 (K), D75.1 (K), D76.1 (K), D77.1 (K)
- net ROW5: now also D78.1 (K), D79.1 (K), D80.1 (K), D81.1 (K), D82.1 (K), D83.1 (K), D84.1 (K), D85.1 (K), D86.1 (K), D87.1 (K), D88.1 (K)
- net VCC: now also C1.1, C2.1, R1.2, R2.2, U1.2 (VCC)
- net SDA: now reaches U2.35 (PC0)
- net SDA: now also R2.1, U1.19 (SDA)
- net SDB: now reaches U2.36 (PC1)
- net SDB: now also R3.1, U1.3 (~SDB)
- net SCL: now reaches U2.37 (PC2)
- net SCL: now also R1.1, U1.20 (SCL)
- net LED1: now reaches U2.38 (PC3)
- net LED1: now also D153.2 (A)
- net LED2: now reaches U2.39 (PC4)
- net LED2: now also D162.2 (A)
- net RGB: no longer names the net of U2.54 (PF7)
- new net: D3.2 (A), MX3.2 (ROW)
- new net: D4.2 (A), MX4.2 (ROW)
- new net: D5.2 (A), MX5.2 (ROW)
- new net: D1.2 (A), MX1.2 (ROW)
- new net: D2.2 (A), MX2.2 (ROW)
- new net: D6.2 (A), MX6.2 (ROW)
- new net: D7.2 (A), MX7.2 (ROW)
- new net: D8.2 (A), MX8.2 (ROW)
- new net: D9.2 (A), MX9.2 (ROW)
- new net: D10.2 (A), MX10.2 (ROW)
- new net: D11.2 (A), MX11.2 (ROW)
- new net: D12.2 (A), MX12.2 (ROW)
- new net: D13.2 (A), MX13.2 (ROW)
- new net: D14.2 (A), MX14.2 (ROW)
- new net: D15.2 (A), MX15.2 (ROW)
- new net: D16.2 (A), MX16.2 (ROW)
- new net: D17.2 (A), MX17.2 (ROW)
- new net: D18.2 (A), MX18.2 (ROW)
- new net: D19.2 (A), MX19.2 (ROW)
- new net: D20.2 (A), MX20.2 (ROW)
- new net: D21.2 (A), MX21.2 (ROW)
- new net: D22.2 (A), MX22.2 (ROW)
- new net: D23.2 (A), MX23.2 (ROW)
- new net: D24.2 (A), MX24.2 (ROW)
- new net: D25.2 (A), MX25.2 (ROW)
- new net: D26.2 (A), MX26.2 (ROW)
- new net: D27.2 (A), MX27.2 (ROW)
- new net: D28.2 (A), MX28.2 (ROW)
- new net: D29.2 (A), MX29.2 (ROW)
- new net: D30.2 (A), MX30.2 (ROW)
- new net: D31.2 (A), MX31.2 (ROW)
- new net: D32.2 (A), MX32.2 (ROW)
- new net: D35.2 (A), MX35.2 (ROW)
- new net: D36.2 (A), MX36.2 (ROW)
- new net: D37.2 (A), MX37.2 (ROW)
- new net: D38.2 (A), MX38.2 (ROW)
- new net: D39.2 (A), MX39.2 (ROW)
- new net: D40.2 (A), MX40.2 (ROW)
- new net: D41.2 (A), MX41.2 (ROW)
- new net: D42.2 (A), MX42.2 (ROW)
- new net: D43.2 (A), MX43.2 (ROW)
- new net: D44.2 (A), MX44.2 (ROW)
- new net: D45.2 (A), MX45.2 (ROW)
- new net: D46.2 (A), MX46.2 (ROW)
- new net: D47.2 (A), MX47.2 (ROW)
- new net: D48.2 (A), MX48.2 (ROW)
- new net: D49.2 (A), MX49.2 (ROW)
- new net: D33.2 (A), MX33.2 (ROW)
- new net: D34.2 (A), MX34.2 (ROW)
- new net: D50.2 (A), MX50.2 (ROW)
- new net: D51.2 (A), MX51.2 (ROW)
- new net: D52.2 (A), MX52.2 (ROW)
- new net: D53.2 (A), MX53.2 (ROW)
- new net: D54.2 (A), MX54.2 (ROW)
- new net: D55.2 (A), MX55.2 (ROW)
- new net: D56.2 (A), MX56.2 (ROW)
- new net: D57.2 (A), MX57.2 (ROW)
- new net: D58.2 (A), MX58.2 (ROW)
- new net: D59.2 (A), MX59.2 (ROW)
- new net: D60.2 (A), MX60.2 (ROW)
- new net: D61.2 (A), MX61.2 (ROW)
- new net: D62.2 (A), MX62.2 (ROW)
- new net: D63.2 (A), MX63.2 (ROW)
- new net: D64.2 (A), MX64.2 (ROW)
- new net: D65.2 (A), MX65.2 (ROW)
- new net: D66.2 (A), MX66.2 (ROW)
- new net: D67.2 (A), MX67.2 (ROW)
- new net: D68.2 (A), MX68.2 (ROW)
- new net: D69.2 (A), MX69.2 (ROW)
- new net: D70.2 (A), MX70.2 (ROW)
- new net: D71.2 (A), MX71.2 (ROW)
- new net: D72.2 (A), MX72.2 (ROW)
- new net: D73.2 (A), MX73.2 (ROW)
- new net: D74.2 (A), MX74.2 (ROW)
- new net: D75.2 (A), MX75.2 (ROW)
- new net: D76.2 (A), MX76.2 (ROW)
- new net: D77.2 (A), MX77.2 (ROW)
- new net: D78.2 (A), MX78.2 (ROW)
- new net: D79.2 (A), MX79.2 (ROW)
- new net: D80.2 (A), MX80.2 (ROW)
- new net: D81.2 (A), MX81.2 (ROW)
- new net: D82.2 (A), MX82.2 (ROW)
- new net: D83.2 (A), MX83.2 (ROW)
- new net: D84.2 (A), MX84.2 (ROW)
- new net: D85.2 (A), MX85.2 (ROW)
- new net: D86.2 (A), MX86.2 (ROW)
- new net: D87.2 (A), MX87.2 (ROW)
- new net: D88.2 (A), MX88.2 (ROW)
- new net: D153.1 (K), R11.2
- new net: D162.1 (K), R12.2
- new net CA1: D105.2 (A), D121.2 (A), D129.2 (A), D137.2 (A), D145.2 (A), D154.2 (A), D163.2 (A), D171.2 (A), D89.1 (K), D90.1 (K), D91.1 (K), D92.1 (K), D93.1 (K), D94.1 (K), D95.1 (K), D96.1 (K), U1.21 (CA1)
- new net CA2: D105.1 (K), D106.1 (K), D107.1 (K), D108.1 (K), D109.1 (K), D110.1 (K), D111.1 (K), D112.1 (K), D122.2 (A), D130.2 (A), D138.2 (A), D146.2 (A), D155.2 (A), D164.2 (A), D172.2 (A), D89.2 (A), U1.22 (CA2)
- new net CA3: D106.2 (A), D121.1 (K), D122.1 (K), D123.1 (K), D124.1 (K), D125.1 (K), D126.1 (K), D127.1 (K), D128.1 (K), D131.2 (A), D139.2 (A), D147.2 (A), D156.2 (A), D165.2 (A), D173.2 (A), D90.2 (A), U1.23 (CA3)
- new net CA4: D107.2 (A), D123.2 (A), D129.1 (K), D130.1 (K), D131.1 (K), D132.1 (K), D133.1 (K), D134.1 (K), D135.1 (K), D136.1 (K), D140.2 (A), D148.2 (A), D157.2 (A), D166.2 (A), D174.2 (A), D91.2 (A), U1.24 (CA4)
- new net CA5: D108.2 (A), D124.2 (A), D132.2 (A), D137.1 (K), D138.1 (K), D139.1 (K), D140.1 (K), D141.1 (K), D142.1 (K), D143.1 (K), D144.1 (K), D149.2 (A), D158.2 (A), D167.2 (A), D175.2 (A), D92.2 (A), U1.25 (CA5)
- new net CA6: D109.2 (A), D125.2 (A), D133.2 (A), D141.2 (A), D145.1 (K), D146.1 (K), D147.1 (K), D148.1 (K), D149.1 (K), D150.1 (K), D151.1 (K), D152.1 (K), D159.2 (A), D168.2 (A), D176.2 (A), D93.2 (A), U1.26 (CA6)
- new net CA7: D110.2 (A), D126.2 (A), D134.2 (A), D142.2 (A), D150.2 (A), D154.1 (K), D155.1 (K), D156.1 (K), D157.1 (K), D158.1 (K), D159.1 (K), D160.1 (K), D161.1 (K), D169.2 (A), D177.2 (A), D94.2 (A), U1.27 (CA7)
- new net CA8: D111.2 (A), D127.2 (A), D135.2 (A), D143.2 (A), D151.2 (A), D160.2 (A), D163.1 (K), D164.1 (K), D165.1 (K), D166.1 (K), D167.1 (K), D168.1 (K), D169.1 (K), D170.1 (K), D178.2 (A), D95.2 (A), U1.28 (CA8)
- new net CA9: D112.2 (A), D128.2 (A), D136.2 (A), D144.2 (A), D152.2 (A), D161.2 (A), D170.2 (A), D171.1 (K), D172.1 (K), D173.1 (K), D174.1 (K), D175.1 (K), D176.1 (K), D177.1 (K), D178.1 (K), D96.2 (A), U1.1 (CA9)
- new net CB1: D100.1 (K), D101.1 (K), D102.1 (K), D103.1 (K), D104.1 (K), D113.1 (K), D113.2 (A), D114.1 (K), D115.1 (K), D116.1 (K), D117.1 (K), D118.1 (K), D119.1 (K), D120.1 (K), D190.2 (A), D97.1 (K), D97.2 (A), D98.1 (K), D99.1 (K), U1.7 (CB1), U1.8 (CB2)
- new net CB3: D114.2 (A), D190.1 (K), D191.1 (K), D191.2 (A), D98.2 (A), U1.9 (CB3)
- new net CB4: D115.2 (A), D99.2 (A), U1.10 (CB4)
- new net CB5: D100.2 (A), D116.2 (A), U1.11 (CB5)
- new net CB6: D101.2 (A), D117.2 (A), U1.12 (CB6)
- new net CB7: D102.2 (A), D118.2 (A), U1.13 (CB7)
- new net CB8: D103.2 (A), D119.2 (A), U1.14 (CB8)
- new net CB9: D104.2 (A), D120.2 (A), U1.15 (CB9)
- new net REXT: R4.2, U1.6 (R_EXT)
- no-connect marks 19 -> 18

Commit message: routing progress
Connections:
- net DN: now reaches R7.2, U3.3 (IO2), USBC1.5 (DN2), USBC1.7 (DN1)
- net DP: now reaches R9.2, U3.2 (IO1), USBC1.6 (DP1), USBC1.8 (DP2)
Changed lines of the file:
@@
 Wire Wire Line
 	5900 6950 5750 6950
+Text GLabel 15550 6000 1    50   Input ~ 0
+DN
+Text GLabel 15550 6100 3    50   Input ~ 0
+DP
 $EndSCHEMATC
