File: keymatrix.sch (KiCad schematic (older format))
At the start: 172 parts

Commit message: annotatedkeyschematic
Parts:
- added D87, D88: D, symbol Device:D
- added MX116: MCRO1, symbol MX_Alps_Hybrid:MX-NoLED
- added MX416: MCRO4, symbol MX_Alps_Hybrid:MX-NoLED
- MX00: value MX-NoLED -> ESC
- MX01: value MX-NoLED -> F1
- MX010: value MX-NoLED -> F10
- MX011: value MX-NoLED -> F11
- MX012: value MX-NoLED -> F12
- MX013: value MX-NoLED -> INSERT
- MX014: value MX-NoLED -> DEL
- MX015: value MX-NoLED -> HOME
- MX02: value MX-NoLED -> F2
- MX03: value MX-NoLED -> F3
- MX04: value MX-NoLED -> F4
- MX05: value MX-NoLED -> F5
- MX06: value MX-NoLED -> F6
- MX07: value MX-NoLED -> F7
- MX08: value MX-NoLED -> F8
- MX09: value MX-NoLED -> F9
- MX10: value MX-NoLED -> ,~
- MX11: value MX-NoLED -> 1!
- MX110: value MX-NoLED -> 0)
- MX111: value MX-NoLED -> -_
- MX112: value MX-NoLED -> =+
- MX114: value MX-NoLED -> BCSP
- MX115: value MX-NoLED -> END
- MX12: value MX-NoLED -> 2@
- MX13: value MX-NoLED -> 3#
- MX14: value MX-NoLED -> 4$
- MX15: value MX-NoLED -> 5%
- MX16: value MX-NoLED -> 6^
- MX17: value MX-NoLED -> 7&
- MX18: value MX-NoLED -> 8*
- MX19: value MX-NoLED -> 9(
- MX20: value MX-NoLED -> TABL
- MX210: value MX-NoLED -> O
- MX211: value MX-NoLED -> P
- MX212: value MX-NoLED -> [{
- MX213: value MX-NoLED -> ]}
- MX214: value MX-NoLED -> \\|
- MX215: value MX-NoLED -> PGUP
- MX216: value MX-NoLED -> MCRO2
- MX22: value MX-NoLED -> Q
- MX23: value MX-NoLED -> W
- MX24: value MX-NoLED -> E
- MX25: value MX-NoLED -> R
- MX26: value MX-NoLED -> T
- MX27: value MX-NoLED -> Y
- MX28: value MX-NoLED -> U
- MX29: value MX-NoLED -> I
- MX30: value MX-NoLED -> CPLK
- MX310: value MX-NoLED -> L
- MX311: value MX-NoLED -> ;:
- MX312: value MX-NoLED -> '\"
- MX313: value MX-NoLED -> ENTR
- MX315: value MX-NoLED -> PGDN
- MX316: value MX-NoLED -> MCRO3
- MX32: value MX-NoLED -> A
- MX33: value MX-NoLED -> S
- MX34: value MX-NoLED -> D
- MX35: value MX-NoLED -> F
- MX36: value MX-NoLED -> G
- MX37: value MX-NoLED -> H
- MX38: value MX-NoLED -> J
- MX39: value MX-NoLED -> K
- MX50: value MX-NoLED -> CTRLL
- MX51: value MX-NoLED -> WIN
- MX510: value MX-NoLED -> ALTR
- MX511: value MX-NoLED -> MENU
- MX512: value MX-NoLED -> FN
- MX513: value MX-NoLED -> CTRLR
- MX514: value MX-NoLED -> LEFT
- MX515: value MX-NoLED -> DOWN
- MX516: value MX-NoLED -> RIGHT
- MX53: value MX-NoLED -> ALTL
- MX56: value MX-NoLED -> SPCB
- Mx41: value MX-NoLED -> SHIFTL
- Mx410: value MX-NoLED -> .>
- Mx411: value MX-NoLED -> /?
- Mx413: value MX-NoLED -> SHIFTR
- Mx415: value MX-NoLED -> UP
- Mx42: value MX-NoLED -> Z
- Mx43: value MX-NoLED -> X
- Mx44: value MX-NoLED -> C
- Mx45: value MX-NoLED -> V
- Mx46: value MX-NoLED -> B
- Mx47: value MX-NoLED -> N
- Mx48: value MX-NoLED -> M
- Mx49: value MX-NoLED -> ,<
Connections:
- net COL16: now also MX116.1 (COL), MX416.1 (COL)
- net ROW1: now also D88.1 (K)
- net ROW4: now also D87.1 (K)
- new net: D87.2 (A), MX416.2 (ROW)
- new net: D88.2 (A), MX116.2 (ROW)

Commit message: maybefinishedschematic
Parts:
- MX013: value INSERT -> HOME
- MX014: value DEL -> END
- MX015: value HOME -> INSERT
- MX115: value END -> DEL
- MX116: value MCRO1 -> MCRO2
- MX216: value MCRO2 -> MCRO3
- MX316: value MCRO3 -> MCRO4
- MX416: value MCRO4 -> MCRO1
Connections:
- net ROW0: now also D87.1 (K)
- net ROW4: no longer D87.1 (K)
Other:
- moved on the sheet: D87, MX416
Changed lines of the file:
@@
 	1    0    0    -1
 $EndComp
-Wire Wire Line
-	10850 3450 10850 4250
 Connection ~ 10250 4250
 Wire Wire Line
@@
 P 10500 3500
 F 0 "MX316" H 10533 3723 60  0000 C CNN
-F 1 "MCRO3" H 10533 3649 20  0000 C CNN
+F 1 "MCRO4" H 10533 3649 20  0000 C CNN
 F 2 "" H 9875 3475 60  0001 C CNN
 F 3 "" H 9875 3475 60  0001 C CNN
@@
 P 10500 2700
 F 0 "MX216" H 10533 2923 60  0000 C CNN
-F 1 "MCRO2" H 10533 2849 20  0000 C CNN
+F 1 "MCRO3" H 10533 2849 20  0000 C CNN
 F 2 "" H 9875 2675 60  0001 C CNN
 F 3 "" H 9875 2675 60  0001 C CNN
@@
 Connection ~ 10850 2650
 Wire Wire Line
-	10850 900  10850 1850
+	10850 900  10850 1050
 Wire Wire Line
 	10250 1850 10250 2650
@@
 P 9900 1900
 F 0 "MX115" H 9933 2123 60  0000 C CNN
-F 1 "END" H 9933 2049 20  0000 C CNN
+F 1 "DEL" H 9933 2049 20  0000 C CNN
 F 2 "" H 9275 1875 60  0001 C CNN
 F 3 "" H 9275 1875 60  0001 C CNN
@@
 P 9900 1100
 F 0 "MX015" H 9933 1323 60  0000 C CNN
-F 1 "HOME" H 9933 1249 20  0000 C CNN
+F 1 "INSERT" H 9933 1249 20  0000 C CNN
 F 2 "" H 9275 1075 60  0001 C CNN
 F 3 "" H 9275 1075 60  0001 C CNN
@@
 P 9300 1100
 F 0 "MX014" H 9333 1323 60  0000 C CNN
-F 1 "DEL" H 9333 1249 20  0000 C CNN
+F 1 "END" H 9333 1249 20  0000 C CNN
 F 2 "" H 8675 1075 60  0001 C CNN
 F 3 "" H 8675 1075 60  0001 C CNN
@@
 P 8700 1100
 F 0 "MX013" H 8733 1323 60  0000 C CNN
-F 1 "INSERT" H 8733 1249 20  0000 C CNN
+F 1 "HOME" H 8733 1249 20  0000 C CNN
 F 2 "" H 8075 1075 60  0001 C CNN
 F 3 "" H 8075 1075 60  0001 C CNN
@@
 $EndComp
 Wire Wire Line
-	10650 4250 10850 4250
+	10650 1050 10850 1050
 $Comp
 L MX_Alps_Hybrid:MX-NoLED MX416
 U 1 1 6551792A
-P 10500 4300
-F 0 "MX416" H 10533 4523 60  0000 C CNN
-F 1 "MCRO4" H 10533 4449 20  0000 C CNN
-F 2 "" H 9875 4275 60  0001 C CNN
-F 3 "" H 9875 4275 60  0001 C CNN
-	1    10500 4300
-	1    0    0    -1
-$EndComp
-Wire Wire Line
-	10450 4750 10450 4800
+P 10500 1100
+F 0 "MX416" H 10533 1323 60  0000 C CNN
+F 1 "MCRO1" H 10533 1249 20  0000 C CNN
+F 2 "" H 9875 1075 60  0001 C CNN
+F 3 "" H 9875 1075 60  0001 C CNN
+	1    10500 1100
+	1    0    0    -1
+$EndComp
+Wire Wire Line
+	10450 1550 10450 1600
 $Comp
 L Device:D D87
 U 1 1 65517935
-P 10450 4600
-F 0 "D87" V 10496 4521 50  0000 R CNN
-F 1 "D" V 10405 4521 50  0000 R CNN
-F 2 "" H 10450 4600 50  0001 C CNN
-F 3 "~" H 10450 4600 50  0001 C CNN
-	1    10450 4600
-	0    -1   -1   0
-$EndComp
-Connection ~ 10850 4250
-Wire Wire Line
-	10850 4250 10850 5050
+P 10450 1400
+F 0 "D87" V 10496 1321 50  0000 R CNN
+F 1 "D" V 10405 1321 50  0000 R CNN
+F 2 "" H 10450 1400 50  0001 C CNN
+F 3 "~" H 10450 1400 50  0001 C CNN
+	1    10450 1400
+	0    -1   -1   0
+$EndComp
 Wire Wire Line
 	10250 4250 10250 5050
 Wire Wire Line
-	10450 4800 9850 4800
-Connection ~ 9850 4800
+	10450 1600 9850 1600
 Wire Wire Line
 	10650 1850 10850 1850
@@
 P 10500 1900
 F 0 "MX116" H 10533 2123 60  0000 C CNN
-F 1 "MCRO1" H 10533 2049 20  0000 C CNN
+F 1 "MCRO2" H 10533 2049 20  0000 C CNN
 F 2 "" H 9875 1875 60  0001 C CNN
 F 3 "" H 9875 1875 60  0001 C CNN
@@
 	10450 2400 9850 2400
 Connection ~ 9850 2400
+Connection ~ 10850 1050
+Wire Wire Line
+	10850 1050 10850 1850
+Wire Wire Line
+	10850 3450 10850 5050
+Connection ~ 9850 1600
 $EndSCHEMATC

Commit message: footprints
Parts:
- D1, D10, D11, D12, D13, D14, D15, D16, D17, D18, D19, D2, D20, D21, D22, D23, D24, D25, D26, D27, D28, D29, D3, D30, D31, D32, D33, D34, D35, D36, D37, D38, D39, D4, D40, D41, D42, D43, D44, D45, D46, D47, D48, D49, D5, D50, D51, D52, D53, D54, D55, D56, D57, D58, D59, D6, D60, D61, D62, D63, D64, D65, D66, D67, D68, D69, D7, D70, D71, D72, D73, D74, D75, D76, D77, D78, D79, D8, D80, D81, D82, D83, D84, D85, D86, D87, D88, D9: footprint (none) -> Diode_SMD:D_SOD-123
- MX00, MX01, MX010, MX011, MX012, MX013, MX014, MX015, MX02, MX03, MX04, MX05, MX06, MX07, MX08, MX09, MX10, MX11, MX110, MX111, MX112, MX115, MX116, MX12, MX13, MX14, MX15, MX16, MX17, MX18, MX19, MX210, MX211, MX212, MX213, MX215, MX216, MX22, MX23, MX24, MX25, MX26, MX27, MX28, MX29, MX310, MX311, MX312, MX315, MX316, MX32, MX33, MX34, MX35, MX36, MX37, MX38, MX39, MX416, MX510, MX511, MX512, MX513, MX514, MX515, MX516, Mx410, Mx411, Mx415, Mx42, Mx43, Mx44, Mx45, Mx46, Mx47, Mx48, Mx49: footprint (none) -> MX_Alps_Hybrid:MX-1U-NoLED
- MX114: footprint (none) -> MX_Alps_Hybrid:MX-2U-NoLED
- MX20, MX214: footprint (none) -> MX_Alps_Hybrid:MX-1.5U-NoLED
- MX30: footprint (none) -> MX_Alps_Hybrid:MX-1.75U-NoLED
- MX313, Mx41: footprint (none) -> MX_Alps_Hybrid:MX-2.25U-NoLED
- MX50, MX51, MX53: footprint (none) -> MX_Alps_Hybrid:MX-1.25U-NoLED
- MX56: footprint (none) -> MX_Alps_Hybrid:MX-6.25U-NoLED
- Mx413: footprint (none) -> MX_Alps_Hybrid:MX-2.75U-NoLED
