File: matrixrgb.sch (KiCad schematic (older format))
At the start: 181 parts

Commit message: nocapschematic
Parts:
- removed C102, C103, C104, C105, C106, C107, C108, C109, C110, C111, C112, C113, C114, C115, C116, C117, C118, C119, C120, C121, C122, C123, C124, C125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: 0.1uF, symbol Device:C_Small
- C101: value 0.1uF -> 100uF
