File: matrix.kicad_pcb (KiCad board)
At the start: 2 copper layers, 48 parts, among them SW1 Rotary_Encoder, SW2 Rotary_Encoder, U1 IS31FL3731-SA, U2 AT90USB1286-AU, U3 PRTR5V0U2X, Y1 16MHz

Commit message: routing progress
Parts:
- moved R5 5.56 mm to (-11.1, 118.3), turned to 0 degrees
- moved U3 5.32 mm to (-39.7, 49.2)
- moved R10 2.78 mm to (-33.3, 52.4), turned to 90 degrees
- moved R6 2.38 mm to (-35.7, 52.4), turned to 90 degrees
- moved Y1 2.12 mm to (-25.4, 115.9)
- moved R12 1.69 mm to (-31.0, 52.4)
- moved R11 0.69 mm to (-47.6, 54.0)
Connections:
- net Net-(R7-Pad2) renamed DN
- net Net-(R9-Pad2) renamed DP
Routing:
- net ROW1: track 0.00 -> 337.3 mm, vias 0 -> 2
- net ROW0: track 0.00 -> 332.7 mm
- net ROW3: track 0.00 -> 323.8 mm, vias 0 -> 2
- net COL3: track 0.00 -> 113.1 mm
- net DN: track 0.00 -> 112.7 mm
- net COL14: track 0.00 -> 112.2 mm
- net DP: track 0.00 -> 110.7 mm
- net COL13: track 0.00 -> 109.7 mm
- net COL10: track 0.00 -> 109.0 mm
- net COL6: track 0.00 -> 108.5 mm
- net COL11: track 0.00 -> 107.9 mm
- net COL1: track 0.00 -> 104.4 mm
- net COL16: track 0.00 -> 103.9 mm
- net COL12: track 0.00 -> 103.5 mm
- net COL15: track 0.00 -> 101.7 mm
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Other:
- board outline added: 354.8 x 125.4 mm
- copper layers 2 -> 4

Commit message: routingcontinue
Parts:
- moved R1 17.7 mm to (160.3, 150.7)
- moved R2 17.4 mm to (158.0, 150.7), turned to 90 degrees
- moved R3 11.6 mm to (158.1, 138.9), turned to 0 degrees
- moved U1 7.32 mm to (148.4, 143.7)
- moved R4 5.56 mm to (157.9, 136.5), turned to 180 degrees
Routing:
- net ROW5: track 0.00 -> 329.8 mm
- net ROW2: track 19.7 -> 326.2 mm
- net ROW4: track 0.00 -> 298.9 mm
- net Net-(D81-Pad2): track 0.00 -> 14.6 mm
- net Net-(D76-Pad2): track 0.00 -> 13.8 mm
- net Net-(D65-Pad2): track 0.00 -> 11.6 mm
- net Net-(D35-Pad2): track 0.00 -> 9.86 mm
- net Net-(D88-Pad2): track 0.00 -> 9.61 mm
- net Net-(D83-Pad2): track 0.00 -> 9.53 mm
- net Net-(D66-Pad2): track 0.00 -> 9.50 mm
- net Net-(D82-Pad2): track 0.00 -> 9.50 mm
- net Net-(D72-Pad2): track 0.00 -> 9.44 mm
- net Net-(D38-Pad2): track 0.00 -> 9.44 mm
- net Net-(D45-Pad2): track 0.00 -> 9.44 mm
- net Net-(D44-Pad2): track 0.00 -> 9.44 mm
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
Commit message: fgvdfuhjkh (final i think)
Parts:
- removed MX81: SPCB, MX_Alps_Hybrid:MX-6.25U-NoLED
- added MX13: F12, MX_Alps_Hybrid:MX-1U-NoLED, B.Cu at (65.1, 50.0)
Routing:
- net CA8: track 0.00 -> 668.6 mm, vias 0 -> 36
- net CA9: track 0.00 -> 648.3 mm, vias 0 -> 27
- net CB1: track 0.00 -> 531.0 mm, vias 0 -> 15
- net CA4: track 0.00 -> 524.4 mm, vias 0 -> 18
- net CA6: track 0.00 -> 510.7 mm, vias 0 -> 18
- net CA7: track 0.00 -> 503.2 mm, vias 0 -> 27
- net CA2: track 0.00 -> 501.5 mm, vias 0 -> 26
- net CA1: track 0.00 -> 496.0 mm, vias 0 -> 17
- net CA5: track 0.00 -> 486.3 mm, vias 0 -> 30
- net CA3: track 0.00 -> 468.6 mm, vias 0 -> 20
- net AD: track 0.00 -> 460.0 mm, vias 0 -> 16
- net COL2: track 0.00 -> 361.8 mm, vias 0 -> 8
- net COL1: track 104.4 -> 454.4 mm, vias 0 -> 2
- net COL0: track 101.6 -> 430.0 mm, vias 0 -> 10
- net VCC: track 0.00 -> 302.1 mm, vias 0 -> 18
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Other:
- copper layers 4 -> 2
