File: attempt2/macropad/macropad.kicad_pcb (KiCad board)
At the start: 2 copper layers, 76.2 x 84.1 mm, 65 parts, among them J1 AVR-ISP-6, SW1 SW_Push, SW2 Rotary_Encoder_Switch, SW3 Rotary_Encoder_Switch, U1 AT90USB1286-AU, Y1 16MHz

Commit message: FinalFinal
Parts:
- U1: value AT90USB1286-AU -> AT90USB1286-MU; footprint Package_QFP:TQFP-64_14x14mm_P0.8mm -> Package_DFN_QFN:QFN-64-1EP_9x9mm_P0.5mm_EP7.5x7.5mm
- moved U1 5.10 mm to (81.1, 70.0)
- moved R4 4.88 mm to (71.6, 65.9), turned to 180 degrees
- moved D1 1.17 mm to (71.0, 76.2), turned to 0 degrees
- moved R3 0.67 mm to (72.9, 63.5), turned to 180 degrees
Routing:
- net GND: track 576.5 -> 561.3 mm, vias 7 -> 5
- net Net-(D1-Pad2): track 35.3 -> 23.9 mm, vias 2 -> 0
- net Net-(SW2-PadB): track 37.1 -> 46.8 mm
- net Net-(SW2-PadA): track 32.1 -> 41.8 mm
- net Net-(SW2-PadS1): track 49.7 -> 59.2 mm
- net Net-(SW3-PadB): track 19.6 -> 29.0 mm
- net Net-(SW3-PadA): track 13.8 -> 23.1 mm
- net Net-(SW3-PadS1): track 24.1 -> 33.2 mm
- net Net-(C2-Pad1): track 9.91 -> 18.6 mm
- net Net-(C3-Pad1): track 16.0 -> 24.7 mm
- net SCK: track 44.0 -> 51.3 mm
- net MOSI: track 44.7 -> 51.2 mm
- net D+: track 12.9 -> 7.22 mm
- net MISO: track 38.3 -> 43.5 mm
- net Row2: track 100.9 -> 106.0 mm
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
Commit message: FullKeebSchematic
Parts:
- U1: value AT90USB1286-MU -> AT90USB1286-AU; footprint Package_DFN_QFN:QFN-64-1EP_9x9mm_P0.5mm_EP7.5x7.5mm -> Package_QFP:TQFP-64_14x14mm_P0.8mm
- moved U1 5.10 mm to (85.7, 72.2)
Connections:
- H1 pad 1: GND -> (no net)
- H2 pad 1: GND -> (no net)
- H3 pad 1: GND -> (no net)
- H4 pad 1: GND -> (no net)
Routing:
- net GND: track 561.3 -> 574.9 mm, vias 5 -> 7
- net Net-(SW2-PadB): track 46.8 -> 37.1 mm
- net Net-(SW2-PadA): track 41.8 -> 32.1 mm
- net Net-(SW2-PadS1): track 59.2 -> 49.7 mm
- net Net-(SW3-PadB): track 29.0 -> 19.6 mm
- net Net-(SW3-PadA): track 23.1 -> 13.8 mm
- net Net-(SW3-PadS1): track 33.2 -> 24.1 mm
- net Net-(C2-Pad1): track 18.6 -> 9.91 mm
- net Net-(C3-Pad1): track 24.7 -> 16.0 mm
- net SCK: track 51.3 -> 44.0 mm
- net MOSI: track 51.2 -> 44.7 mm
- net D+: track 7.22 -> 12.5 mm
- net MISO: track 43.5 -> 38.3 mm
- net Row2: track 106.0 -> 100.9 mm
- net Col3: track 85.7 -> 80.6 mm
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