File: attempt2/macropad/macropad.sch (KiCad schematic (older format))
At the start: 65 parts, among them J1 AVR-ISP-6, SW1 SW_Push, SW2 Rotary_Encoder_Switch, SW3 Rotary_Encoder_Switch, U1 AT90USB1286-AU, Y1 16MHz

Commit message: FinalFinal
Parts:
- removed U1: AT90USB1286-AU, Package_QFP:TQFP-64_14x14mm_P0.8mm, symbol MCU_Microchip_AVR:AT90USB1286-AU
- added U1: AT90USB1286-MU, Package_DFN_QFN:QFN-64-1EP_9x9mm_P0.5mm_EP7.5x7.5mm, symbol MCU_Microchip_AVR:AT90USB1286-MU
Changed lines of the file:
@@
 Wire Wire Line
 	9800 6950 9800 6750
-Connection ~ 8000 7800
-Wire Wire Line
-	8000 7800 7950 7800
-Wire Wire Line
-	8100 7800 8000 7800
-Connection ~ 8000 3800
-Connection ~ 8100 3800
-Wire Wire Line
-	8100 3800 8200 3800
-Wire Wire Line
-	8000 3800 8100 3800
 Wire Wire Line
 	8750 7550 8750 7400
-$Comp
-L MCU_Microchip_AVR:AT90USB1286-AU U1
-U 1 1 65FA2E75
-P 8100 5800
-F 0 "U1" H 8100 3711 50  0000 C CNN
-F 1 "AT90USB1286-AU" H 8100 3620 50  0000 C CNN
-F 2 "Package_QFP:TQFP-64_14x14mm_P0.8mm" H 8100 5800 50  0001 C CIN
-F 3 "http://ww1.microchip.com/downloads/en/DeviceDoc/doc7593.pdf" H 8100 5800 50  0001 C CNN
-	1    8100 5800
-	1    0    0    -1
-$EndComp
 Wire Wire Line
 	9050 7100 9050 6950
@@
 	1    0    0    -1
 $EndComp
+Wire Wire Line
+	8000 3800 8100 3800
+Wire Wire Line
+	7950 7800 8000 7800
+$Comp
+L MCU_Microchip_AVR:AT90USB1286-MU U1
+U 1 1 65FFB91E
+P 8100 5800
+F 0 "U1" H 8100 3711 50  0000 C CNN
+F 1 "AT90USB1286-MU" H 8100 3620 50  0000 C CNN
+F 2 "Package_DFN_QFN:QFN-64-1EP_9x9mm_P0.5mm_EP7.5x7.5mm" H 8100 5800 50  0001 C CIN
+F 3 "http://ww1.microchip.com/downloads/en/DeviceDoc/doc7593.pdf" H 8100 5800 50  0001 C CNN
+	1    8100 5800
+	1    0    0    -1
+$EndComp
+Connection ~ 8000 3800
+Wire Wire Line
+	8100 3800 8200 3800
+Connection ~ 8100 3800
+Wire Wire Line
+	8000 7800 8100 7800
+Connection ~ 8000 7800
 $EndSCHEMATC

Commit message: FullKeebSchematic
Parts:
- removed C1: 1uF, Capacitor_SMD:C_0805_2012Metric, symbol Device:C_Small
- removed C2, C3: 22pF, Capacitor_SMD:C_0805_2012Metric, symbol Device:C_Small
- removed C4: 10uF, Capacitor_SMD:C_0805_2012Metric, symbol Device:C_Small
- removed C5, C6, C7, C8, C9: 0.1uF, Capacitor_SMD:C_0805_2012Metric, symbol Device:C_Small
- removed D1: PRTR5V0U2X, Package_TO_SOT_SMD:SOT-143, symbol Power_Protection:PRTR5V0U2X
- removed D10, D11, D12, D13, D2, D3, D4, D5, D6, D7, D8, D9: SK6812MINI-E, kicad-keyboard-parts:MX_SK6812MINI-E, symbol kicad-keyboard-parts:SK6812MINI-E
- removed D14, D15, D16, D17, D18, D19, D20, D21, D22, D23, D24, D25: D_Small, Diode_SMD:D_SOD-123, symbol Device:D_Small
- removed F1: 500m, Fuse:Fuse_1206_3216Metric_Pad1.42x1.75mm_HandSolder, symbol Device:Polyfuse_Small
- removed H1, H2, H3, H4: MountingHole, MountingHole:MountingHole_2.2mm_M2_DIN965_Pad, symbol Mechanical:MountingHole
- removed J1: AVR-ISP-6, random-keyboard-parts:Reset_Pretty-Mask, symbol Connector:AVR-ISP-6
- removed MX1, MX10, MX11, MX12, MX2, MX3, MX4, MX5, MX6, MX7, MX8, MX9: MX-NoLED, MX_Only:MXOnly-1U-NoLED, symbol MX_Alps_Hybrid:MX-NoLED
- removed R1, R2: 5.1k, Resistor_SMD:R_0805_2012Metric, symbol Device:R_Small_US
- removed R3, R4: 22, Resistor_SMD:R_0805_2012Metric, symbol Device:R_Small_US
- removed R5: 1k, Resistor_SMD:R_0805_2012Metric, symbol Device:R_Small_US
- removed R6: 10k, Resistor_SMD:R_0805_2012Metric, symbol Device:R_Small_US
- removed R7: 499, Resistor_SMD:R_0805_2012Metric, symbol Device:R_Small_US
- removed SW1: SW_Push, random-keyboard-parts:SKQG-1155865, symbol Switch:SW_Push
- removed SW2, SW3: Rotary_Encoder_Switch, Rotary_Encoder:RotaryEncoder_Alps_EC11E-Switch_Vertical_H20mm, symbol Device:Rotary_Encoder_Switch
- removed U1: AT90USB1286-MU, Package_DFN_QFN:QFN-64-1EP_9x9mm_P0.5mm_EP7.5x7.5mm, symbol MCU_Microchip_AVR:AT90USB1286-MU
- removed USB1: HRO-TYPE-C-31-M-12, Type-C:HRO-TYPE-C-31-M-12-HandSoldering, symbol Type-C:HRO-TYPE-C-31-M-12
- removed Y1: 16MHz, Crystal:Crystal_SMD_3225-4Pin_3.2x2.5mm, symbol Device:Crystal_GND24_Small
Connections:
- no-connect marks 33 -> 0
