File: keyboard/keeb.kicad_pcb (KiCad board)
At the start: 4 copper layers, 390.5 x 126.2 mm, 330 parts, among them J1 AVR-ISP-6, SW1 SW_Push, SW3 Rotary_Encoder_Switch, SW4 Rotary_Encoder_Switch, SW5 Rotary_Encoder_Switch, U1 AT90USB1286-MU, Y1 16MHz

Commit message: keeb-fillzones
Routing:
- net +5V: track 2557.5 -> 2580.0 mm, vias 10 -> 14
- added copper zone on In1.Cu, net +5V
- added copper zone on In2.Cu, net GND
Changed lines of the file:
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@@
     (thickness 1.6)
     (drawings 27)
-    (tracks 2710)
+    (tracks 2725)
     (zones 0)
     (modules 330)
@@
   (segment (start 290.29375 91.926249) (end 290.29375 92.436249) (width 0.385) (layer B.Cu) (net 5))
   (segment (start 291.118464 91.101535) (end 290.29375 91.926249) (width 0.385) (layer B.Cu) (net 5))
-  (segment (start 312.771536 91.101535) (end 291.118464 91.101535) (width 0.385) (layer B.Cu) (net 5))
   (segment (start 314.10625 92.436249) (end 312.771536 91.101535) (width 0.385) (layer B.Cu) (net 5))
   (segment (start 271.24375 91.926249) (end 271.24375 92.436249) (width 0.385) (layer B.Cu) (net 5))
@@
   (segment (start 371.261249 76.2) (end 370.10625 75.045001) (width 0.385) (layer B.Cu) (net 5))
   (segment (start 397.45 79.736249) (end 393.913751 76.2) (width 0.385) (layer B.Cu) (net 5))
-  (segment (start 393.913751 76.2) (end 371.261249 76.2) (width 0.385) (layer B.Cu) (net 5))
   (segment (start 227.90054 130.055539) (end 228.38125 130.536249) (width 0.385) (layer B.Cu) (net 5))
   (segment (start 226.436652 128.591651) (end 227.90054 130.055539) (width 0.385) (layer B.Cu) (net 5))
@@
   (segment (start 398.862499 105.968749) (end 401.53279 105.968749) (width 0.385) (layer In2.Cu) (net 5))
   (segment (start 398.4625 105.56875) (end 398.862499 105.968749) (width 0.385) (layer In2.Cu) (net 5))
+  (via (at 382.5875 76.99375) (size 0.8) (drill 0.4) (layers F.Cu B.Cu) (net 5))
+  (segment (start 383.38125 76.2) (end 382.5875 76.99375) (width 0.385) (layer B.Cu) (net 5))
+  (segment (start 383.38125 76.2) (end 371.261249 76.2) (width 0.385) (layer B.Cu) (net 5))
+  (segment (start 393.913751 76.2) (end 383.38125 76.2) (width 0.385) (layer B.Cu) (net 5))
+  (segment (start 312.771536 91.101535) (end 291.118464 91.101535) (width 0.385) (layer B.Cu) (net 5))
+  (via (at 268.2875 92.075) (size 0.8) (drill 0.4) (layers F.Cu B.Cu) (net 5))
+  (segment (start 269.909036 91.101535) (end 269.260965 91.101535) (width 0.385) (layer B.Cu) (net 5))
+  (segment (start 269.260965 91.101535) (end 268.2875 92.075) (width 0.385) (layer B.Cu) (net 5))
+  (via (at 302.41875 84.93125) (size 0.8) (drill 0.4) (layers F.Cu B.Cu) (net 5))
+  (segment (start 314.10625 92.436249) (end 309.923749 92.436249) (width 0.385) (layer B.Cu) (net 5))
+  (segment (start 309.923749 92.436249) (end 302.41875 84.93125) (width 0.385) (layer B.Cu) (net 5))
+  (segment (start 314.475046 92.291905) (end 314.473779 92.259501) (width 0.385) (layer B.Cu) (net 5))
+  (segment (start 314.10625 92.436249) (end 314.330702 92.436249) (width 0.385) (layer B.Cu) (net 5))
+  (segment (start 314.330702 92.436249) (end 314.475046 92.291905) (width 0.385) (layer B.Cu) (net 5))
+  (via (at 342.9 89.69375) (size 0.8) (drill 0.4) (layers F.Cu B.Cu) (net 5))
+  (segment (start 345.85625 92.436249) (end 343.113751 89.69375) (width 0.385) (layer B.Cu) (net 5))
+  (segment (start 343.113751 89.69375) (end 342.9 89.69375) (width 0.385) (layer B.Cu) (net 5))
   (segment (start 392.975 42.589172) (end 392.975 43.91375) (width 0.385) (layer B.Cu) (net 6))
   (segment (start 391.660828 41.275) (end 392.975 42.589172) (width 0.385) (layer B.Cu) (net 6))
@@
   (segment (start 334.529999 130.536249) (end 307.4 130.536249) (width 0.25) (layer B.Cu) (net 246))
   (segment (start 343.967499 139.973749) (end 334.529999 130.536249) (width 0.25) (layer B.Cu) (net 246))
+  (zone (net 5) (net_name +5V) (layer In1.Cu) (hatch edge 0.508)
+    (connect_pads (clearance 0.508))
+    (min_thickness 0.254)
+    (fill yes (arc_segments 32) (thermal_gap 0.508) (thermal_bridge_width 0.508))
+    (polygon
+      (pts
+        (xy -98.425 -40.48125) (xy 508.79375 -27.78125) (xy 517.525 283.36875) (xy -63.5 260.35)
+      )
+    )
+  )
+  (zone (net 1) (net_name GND) (layer In2.Cu) (hatch edge 0.508)
+    (connect_pads (clearance 0.508))
+    (min_thickness 0.254)
+    (fill yes (arc_segments 32) (thermal_gap 0.508) (thermal_bridge_width 0.508))
+    (polygon
+      (pts
+        (xy 473.075 19.05) (xy -30.1625 11.1125) (xy -8.73125 196.05625) (xy 446.0875 215.9)
+      )
+    )
+  )
 )

Commit message: It works
Works ╰(*°▽°*)╯
Parts:
- removed D103: D_Small, Diode_SMD:D_SOD-123
- removed D201: SK6812MINI-E, kicad-keyboard-parts:MX_SK6812MINI-E
- removed MX91: MX-NoLED, MX_Only:MXOnly-1U-NoLED
- MX84, MX90: footprint MX_Only:MXOnly-1U-NoLED -> MX_Only:MXOnly-1.25U-NoLED
- moved D102 4.76 mm to (285.8, 138.9)
- moved D200 4.76 mm to (292.9, 155.6)
- moved MX90 4.76 mm to (292.9, 145.3)
- moved D104 3.18 mm to (322.3, 146.9)
- moved D105 3.18 mm to (341.3, 146.9)
- moved D106 3.18 mm to (360.4, 146.9)
- moved D184 3.18 mm to (348.5, 134.1)
- moved D202 3.18 mm to (329.4, 163.5)
- moved D203 3.18 mm to (348.5, 163.5)
- moved D94 3.18 mm to (341.3, 127.8)
- moved H10 3.18 mm to (331.0, 138.9)
- moved MX82 3.18 mm to (348.5, 134.1)
- moved MX92 3.18 mm to (329.4, 153.2)
- moved MX93 3.18 mm to (348.5, 153.2)
- moved D204 3.17 mm to (367.5, 163.5)
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Connections:
- D202 pad 4: Net-(D201-Pad2) -> Net-(D200-Pad2)
Routing:
- net Col15: track 214.9 -> 174.9 mm
- net Net-(D201-Pad2): track 24.1 -> 0.00 mm
- net Net-(D200-Pad2): track 14.5 -> 35.2 mm
- net GND: track 2627.1 -> 2612.3 mm
- net +5V: track 2580.0 -> 2569.7 mm
- net Net-(D63-Pad2): track 0.00 -> 9.87 mm
- net Net-(D62-Pad2): track 0.00 -> 9.87 mm
- net Net-(D103-Pad2): track 9.84 -> 0.00 mm
- net Net-(D183-Pad4): track 45.5 -> 42.4 mm
- net Net-(D169-Pad2): track 46.7 -> 49.9 mm
- net Row2: track 413.0 -> 415.8 mm
- net Net-(D199-Pad2): track 16.9 -> 19.2 mm
- net Col4: track 407.9 -> 410.3 mm
- net Net-(D189-Pad2): track 22.4 -> 24.8 mm
- net Col3: track 433.4 -> 435.8 mm
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Other:
- outline, holes or cut-outs redrawn
