File: keyboard/keeb.sch (KiCad schematic (older format))
At the start: 337 parts, among them J1 AVR-ISP-6, SW1 SW_Push, SW3 Rotary_Encoder_Switch, SW4 Rotary_Encoder_Switch, SW5 Rotary_Encoder_Switch, U1 AT90USB1286-MU, Y1 16MHz

Commit message: keeb-routed
Parts:
- removed D170, D185, D186, D187, D188, D205, D206: SK6812MINI-E, kicad-keyboard-parts:MX_SK6812MINI-E, symbol kicad-keyboard-parts:SK6812MINI-E
- MX10, MX50: footprint MX_Only:MXOnly-1U-NoLED -> MX_Only:MXOnly-1.5U-NoLED
- MX37: footprint MX_Only:MXOnly-1U-NoLED -> MX_Only:MXOnly-2U-NoLED
- MX54: footprint MX_Only:MXOnly-1U-NoLED -> MX_Only:MXOnly-1.75U-NoLED
- MX66, MX70: footprint MX_Only:MXOnly-1U-NoLED -> MX_Only:MXOnly-2.25U-NoLED
- MX81: footprint MX_Only:MXOnly-1U-NoLED -> MX_Only:MXOnly-2.75U-NoLED
- MX85, MX86, MX88, MX89: footprint MX_Only:MXOnly-1U-NoLED -> MX_Only:MXOnly-1.25U-NoLED
- MX87: footprint MX_Only:MXOnly-1U-NoLED -> MX_Only:MXOnly-6.25U-NoLED
Connections:
- net Col1: no longer D22.1 (K), D23.1 (K), D24.1 (K), D25.1 (K), D50.1 (K), D51.1 (K), D52.1 (K), D53.1 (K), D54.1 (K), D55.1 (K), D56.1 (K), D57.1 (K), D58.1 (K), D59.1 (K), D60.1 (K), D62.1 (K), D63.1 (K), MX10.1 (COL), MX11.1 (COL), MX13.1 (COL), MX14.1 (COL), MX15.1 (COL), MX17.1 (COL), MX18.1 (COL), MX19.1 (COL), MX2.1 (COL), MX21.1 (COL), MX22.1 (COL), MX23.1 (COL), MX25.1 (COL), MX26.1 (COL), MX27.1 (COL), MX28.1 (COL), MX29.1 (COL), MX3.1 (COL), MX31.1 (COL), MX32.1 (COL), MX33.1 (COL), MX35.1 (COL), MX36.1 (COL), MX37.1 (COL), MX38.1 (COL), MX39.1 (COL), MX40.1 (COL), MX41.1 (COL), MX42.1 (COL), MX44.1 (COL), MX45.1 (COL), MX46.1 (COL), MX48.1 (COL), MX49.1 (COL), MX50.1 (COL), MX51.1 (COL), MX52.1 (COL), MX54.1 (COL), MX56.1 (COL), MX57.1 (COL), MX58.1 (COL), MX6.1 (COL), MX60.1 (COL), MX61.1 (COL), MX62.1 (COL), MX64.1 (COL), MX65.1 (COL), MX66.1 (COL), MX67.1 (COL), MX68.1 (COL), MX7.1 (COL), MX70.1 (COL), MX72.1 (COL), MX73.1 (COL), MX74.1 (COL), MX76.1 (COL), MX77.1 (COL), MX78.1 (COL), MX80.1 (COL), MX81.1 (COL), MX82.1 (COL), MX84.1 (COL), MX85.1 (COL), MX89.1 (COL), MX90.1 (COL), MX91.1 (COL), MX93.1 (COL), MX94.1 (COL), U1.10 (PB0), U1.11 (PB1), U1.12 (PB2), U1.14 (PB4), U1.15 (PB5), U1.16 (PB6), U1.35 (PC0), U1.36 (PC1), U1.40 (PC5), U1.45 (PA6), U1.46 (PA5), U1.47 (PA4), U1.49 (PA2), U1.50 (PA1)
- net GND: now also D204.2 (DOUT); no longer D189.4 (DIN)
- net MISO: now also U1.36 (PC1); no longer U1.18 (PE4)
- net MOSI: now also U1.35 (PC0); no longer U1.19 (PE5)
- net Row3: now also D78.1 (K)
- net Row5: now also D46.1 (K)
- net at R7.1: now also D116.4 (DIN); no longer D2.4 (DIN)
- net at D3.2 (DOUT): now also D2.4 (DIN); no longer D4.4 (DIN)
- net at D3.4 (DIN): now also D4.2 (DOUT); no longer D2.2 (DOUT)
- net at D5.4 (DIN): now also D6.2 (DOUT); no longer D4.2 (DOUT)
- net at D5.2 (DOUT): now also D4.4 (DIN); no longer D6.4 (DIN)
- net at D7.4 (DIN): now also D8.2 (DOUT); no longer D6.2 (DOUT)
- net at D7.2 (DOUT): now also D6.4 (DIN); no longer D8.4 (DIN)
- net at D9.4 (DIN): now also D107.2 (DOUT); no longer D8.2 (DOUT)
- net at D9.2 (DOUT): now also D8.4 (DIN); no longer D107.4 (DIN)
- net at D108.4 (DIN): now also D109.2 (DOUT); no longer D107.2 (DOUT)
- net at D108.2 (DOUT): now also D107.4 (DIN); no longer D109.4 (DIN)
- net at D110.4 (DIN): now also D111.2 (DOUT); no longer D109.2 (DOUT)
- net at D110.2 (DOUT): now also D109.4 (DIN); no longer D111.4 (DIN)
- net at D112.2 (DOUT): now also D111.4 (DIN); no longer D113.4 (DIN)
- net at D112.4 (DIN): now also D113.2 (DOUT); no longer D111.2 (DOUT)
- net at D114.2 (DOUT): now also D113.4 (DIN); no longer D115.4 (DIN)
- net at D114.4 (DIN): now also D115.2 (DOUT); no longer D113.2 (DOUT)
- net at D116.2 (DOUT): now also D115.4 (DIN); no longer D134.2 (DOUT)
- net at D117.4 (DIN): now also D2.2 (DOUT); no longer D135.4 (DIN)
- net at D135.2 (DOUT): now also D153.4 (DIN); no longer D136.4 (DIN)
- net at D136.2 (DOUT): now also D135.4 (DIN); no longer D137.4 (DIN)
- net at D137.2 (DOUT): now also D136.4 (DIN); no longer D138.4 (DIN)
- net at D138.2 (DOUT): now also D137.4 (DIN); no longer D139.4 (DIN)
- net at D140.2 (DOUT): now also D139.4 (DIN); no longer D141.4 (DIN)
- net at D139.2 (DOUT): now also D138.4 (DIN); no longer D140.4 (DIN)
- net at D142.2 (DOUT): now also D141.4 (DIN); no longer D143.4 (DIN)
- net at D141.2 (DOUT): now also D140.4 (DIN); no longer D142.4 (DIN)
- net at D143.2 (DOUT): now also D142.4 (DIN); no longer D144.4 (DIN)
- net at D144.2 (DOUT): now also D143.4 (DIN); no longer D145.4 (DIN)
- net at D145.2 (DOUT): now also D144.4 (DIN); no longer D146.4 (DIN)
- net at D146.2 (DOUT): now also D145.4 (DIN); no longer D147.4 (DIN)
- net at D148.2 (DOUT): now also D147.4 (DIN); no longer D149.4 (DIN)
- net at D147.2 (DOUT): now also D146.4 (DIN); no longer D148.4 (DIN)
- net at D150.2 (DOUT): now also D149.4 (DIN); no longer D151.4 (DIN)
- net at D149.2 (DOUT): now also D148.4 (DIN); no longer D150.4 (DIN)
- net at D152.2 (DOUT): now also D151.4 (DIN)
- net at D152.4 (DIN): now also D134.2 (DOUT); no longer D151.2 (DOUT)
- net at D171.4 (DIN): now also D172.2 (DOUT); no longer D153.4 (DIN)
- net at D169.2 (DOUT): now also D184.4 (DIN)
- net at D171.2 (DOUT): now also D189.4 (DIN); no longer D172.4 (DIN)
- net at D173.4 (DIN): now also D174.2 (DOUT); no longer D172.2 (DOUT)
- net at D173.2 (DOUT): now also D172.4 (DIN); no longer D174.4 (DIN)
- net at D175.4 (DIN): now also D176.2 (DOUT); no longer D174.2 (DOUT)
- net at D177.4 (DIN): now also D178.2 (DOUT); no longer D176.2 (DOUT)
- net at D175.2 (DOUT): now also D174.4 (DIN); no longer D176.4 (DIN)
- net at D179.4 (DIN): now also D180.2 (DOUT); no longer D178.2 (DOUT)
- net at D177.2 (DOUT): now also D176.4 (DIN); no longer D178.4 (DIN)
- net at D179.2 (DOUT): now also D178.4 (DIN); no longer D180.4 (DIN)
- net at D181.4 (DIN): now also D182.2 (DOUT); no longer D180.2 (DOUT)
- net at D181.2 (DOUT): now also D180.4 (DIN); no longer D182.4 (DIN)
- net at D183.4 (DIN): now also D184.2 (DOUT); no longer D182.2 (DOUT)
- net at D183.2 (DOUT): now also D182.4 (DIN); no longer D184.4 (DIN)
- net Row4: now reaches D61.1 (K)
- net Row4: now also D22.1 (K), D23.1 (K), D24.1 (K), D25.1 (K), D50.1 (K), D51.1 (K), D52.1 (K), D53.1 (K), D54.1 (K), D55.1 (K), D56.1 (K), D57.1 (K), D58.1 (K), D59.1 (K), D60.1 (K), D62.1 (K), D63.1 (K), U1.40 (PC5)
- new net: D150.4 (DIN), D151.2 (DOUT)
- new net Col10: MX18.1 (COL), MX32.1 (COL), MX45.1 (COL), MX61.1 (COL), MX77.1 (COL), U1.11 (PB1)
- new net Col11: MX19.1 (COL), MX33.1 (COL), MX46.1 (COL), MX62.1 (COL), MX78.1 (COL), U1.12 (PB2)
- new net Col13: MX21.1 (COL), MX35.1 (COL), MX48.1 (COL), MX64.1 (COL), MX80.1 (COL), MX89.1 (COL), U1.14 (PB4)
- new net Col14: MX22.1 (COL), MX36.1 (COL), MX49.1 (COL), MX65.1 (COL), MX81.1 (COL), MX90.1 (COL), U1.15 (PB5)
- new net Col15: MX23.1 (COL), MX37.1 (COL), MX50.1 (COL), MX66.1 (COL), MX91.1 (COL), U1.16 (PB6)
- new net Col17: MX25.1 (COL), MX38.1 (COL), MX51.1 (COL), MX67.1 (COL), MX82.1 (COL), MX93.1 (COL), U1.18 (PE4)
- new net Col18: MX26.1 (COL), MX39.1 (COL), MX52.1 (COL), MX68.1 (COL), MX94.1 (COL), U1.19 (PE5)
- new net Col2: MX10.1 (COL), MX2.1 (COL), MX54.1 (COL), MX6.1 (COL), MX70.1 (COL), MX84.1 (COL), U1.50 (PA1)
- new net Col3: MX11.1 (COL), MX3.1 (COL), MX7.1 (COL), MX85.1 (COL), U1.49 (PA2)
- new net Col5: MX13.1 (COL), MX27.1 (COL), MX40.1 (COL), MX56.1 (COL), MX72.1 (COL), U1.47 (PA4)
- new net Col6: MX14.1 (COL), MX28.1 (COL), MX41.1 (COL), MX57.1 (COL), MX73.1 (COL), U1.46 (PA5)
- new net Col7: MX15.1 (COL), MX29.1 (COL), MX42.1 (COL), MX58.1 (COL), MX74.1 (COL), U1.45 (PA6)
- new net Col9: MX17.1 (COL), MX31.1 (COL), MX44.1 (COL), MX60.1 (COL), MX76.1 (COL), U1.10 (PB0)
Other:
- moved on the sheet: C2, C3, C4, C5, C6, C7, C8, C9, D10, D100, D101, D102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

Commit message: It works
Works ╰(*°▽°*)╯
Parts:
- removed D103: D_Small, Diode_SMD:D_SOD-123, symbol Device:D_Small
- removed D201: SK6812MINI-E, kicad-keyboard-parts:MX_SK6812MINI-E, symbol kicad-keyboard-parts:SK6812MINI-E
- removed MX91: MX-NoLED, MX_Only:MXOnly-1U-NoLED, symbol MX_Alps_Hybrid:MX-NoLED
- MX84, MX90: footprint MX_Only:MXOnly-1U-NoLED -> MX_Only:MXOnly-1.25U-NoLED
Connections:
- net at D200.2 (DOUT): now also D202.4 (DIN)
Other:
- moved on the sheet: D202, D203, D204
